File: MainBoardV3/Power sheet.kicad_sch (KiCad schematic)
At the start: 21 parts, among them J12 Conn_01x02, J13 Conn_01x02, J14 Conn_01x02, J15 Conn_01x02, J16 Conn_01x02, J17 Conn_01x02, J6 Conn_01x02, U1 TSR_2-2450, U3 TSR_2-2433, U4 TEN_50-2411WI

Commit message: Modified to suit needs
Parts:
- removed C1, C2, C4: C_Polarized, Capacitor_THT:CP_Radial_D5.0mm_P2.50mm, symbol Device:C_Polarized
- removed C3: C_Polarized, Capacitor_THT:CP_Radial_D8.0mm_P3.80mm, symbol Device:C_Polarized
- removed C5: C_Polarized, Capacitor_THT:CP_Radial_D8.0mm_P3.50mm, symbol Device:C_Polarized
- removed D4 (x3): LED_Small, LED_SMD:LED_1206_3216Metric_Pad1.42x1.75mm_HandSolder, symbol Device:LED_Small
- removed R5 (x3): R_Small, Resistor_SMD:R_1206_3216Metric_Pad1.30x1.75mm_HandSolder, symbol Device:R_Small
- removed U1: TSR_2-2450, Traco:Traco 2- 24xx, symbol Traco:TSR_2-2450
- removed U3: TSR_2-2433, Traco:Traco 2- 24xx, symbol Traco:TSR_2-2433
- removed U4: TEN_50-2411WI, Traco:Traco TEN 50 series, symbol Traco:TEN_50-2411WI
Connections:
- no-connect marks 1 -> 0
