File: MainBoardV3/MainboardV3.kicad_pcb (KiCad board)
At the start: 2 copper layers, 100 x 100 mm, 53 parts, among them J1 Conn_01x02, J10 Conn_01x04, J11 Conn_01x02, J12 Conn_01x02, J13 Conn_01x02, J14 Conn_01x02, J15 Conn_01x02, J16 Conn_01x02, J17 Conn_01x02, J18 Conn_01x03, J19 Conn_02x03_Odd_Even, J2 Conn_01x04, J20 Conn_02x03_Odd_Even, J21 Conn_02x03_Odd_Even, J22 Conn_01x03, J23 Conn_01x05, J24 Conn_02x05_Odd_Even, J3 Conn_01x03, J4 Conn_01x04, J5 Conn_01x05, J6 Conn_01x02, J7 Conn_01x04, J8 Conn_01x04, J9 Conn_01x04, U1 TSR_2-2450, U2 ESP32-S3-DevKitC, U3 TSR_2-2433, U4 TEN_50-2411WI

Commit message: Adapted schematic to existing needs
Parts:
- removed A1, A2, A3: Pololu_Breakout_DRV8825, Module:Pololu_Breakout-16_15.2x20.3mm
- removed C4: C_Polarized, Capacitor_THT:CP_Radial_D5.0mm_P2.50mm
- removed C5, C7, C8, C9: C_Polarized, Capacitor_THT:CP_Radial_D8.0mm_P3.50mm
- removed D1, D3, D4: LED_Small, LED_SMD:LED_1206_3216Metric_Pad1.42x1.75mm_HandSolder
- removed J10, J2, J4: Conn_01x04, Connector_Molex:Molex_KK-254_AE-6410-04A_1x04_P2.54mm_Vertical
- removed J11, Tir.1: Conn_01x02, Connector_JST:JST_XH_B2B-XH-A_1x02_P2.50mm_Vertical
- removed J12, J13, J14, J15, J16, J17: Conn_01x02, Connector_Molex:Molex_KK-254_AE-6410-02A_1x02_P2.54mm_Vertical
- removed J18, J22, J3: Conn_01x03, Connector_PinHeader_2.54mm:PinHeader_1x03_P2.54mm_Vertical
- removed J19, J20, J21: Conn_02x03_Odd_Even, Connector_PinHeader_2.54mm:PinHeader_2x03_P2.54mm_Vertical
- removed J23, J5: Conn_01x05, Connector_JST:JST_XH_B5B-XH-A_1x05_P2.50mm_Vertical
- removed J24: Conn_02x05_Odd_Even, Connector_IDC:IDC-Header_2x05_P2.54mm_Vertical
- removed J6: Conn_01x02, Connector_AMASS:AMASS_XT60-M_1x02_P7.20mm_Vertical
- removed J7, J8, J9: Conn_01x04, Connector_JST:JST_XH_B4B-XH-A_1x04_P2.50mm_Vertical
- removed U2: ESP32-S3-DevKitC, ESP:ESP32-S3-DevKitC
- removed U3: TSR_2-2433, Traco:Traco 2- 24xx
- removed U4: TEN_50-2411WI, Traco:Traco TEN 50 series
- removed U5: ~, Custom:PCA9685breakout
- added Conn12V1: Conn12V, Connector_AMASS:AMASS_XT30U-F_1x02_P5.0mm_Vertical, F.Cu at (322.5, 187.8)
- added Conn5V1: Conn5V, Connector_Molex:Molex_KK-254_AE-6410-02A_1x02_P2.54mm_Vertical, F.Cu at (132.5, 92.2)
- added Conn5VL1: Conn5VL, Connector_Molex:Molex_KK-254_AE-6410-02A_1x02_P2.54mm_Vertical, F.Cu at (137.7, 72.3)
- added Conn5VP1: Conn5VP, Connector_Molex:Molex_KK-396_A-41791-0002_1x02_P3.96mm_Vertical, F.Cu at (164.5, 111.6)
- added ConnAfficheur1: ConnAfficheur, Connector_JST:JST_EH_B6B-EH-A_1x06_P2.50mm_Vertical, F.Cu at (138.8, 90.8)
- added ConnBATT1: ConnBATT, Connector_AMASS:AMASS_XT60-F_1x02_P7.20mm_Vertical, F.Cu at (322.8, 143.0)
- added ConnButton2: ConnButton2, Connector_Molex:Molex_KK-254_AE-6410-02A_1x02_P2.54mm_Vertical, F.Cu at (166.2, 62.3)
- added ConnButton3: ConnButton3, Connector_Molex:Molex_KK-254_AE-6410-02A_1x02_P2.54mm_Vertical, F.Cu at (166.5, 52.0)
- added ConnI2C1: ConnI2C, Connector_Molex:Molex_KK-254_AE-6410-03A_1x03_P2.54mm_Vertical, F.Cu at (130.5, 80.2)
- added ConnIFM_1: ConnIFM_1, Connector_Molex:Molex_KK-254_AE-6410-03A_1x03_P2.54mm_Vertical, F.Cu at (317.4, 163.3)
- added ConnIFM_2: ConnIFM_2, Connector_Molex:Molex_KK-254_AE-6410-03A_1x03_P2.54mm_Vertical, F.Cu at (317.4, 171.2)
- added ConnIFM_3: ConnIFM_3, Connector_Molex:Molex_KK-254_AE-6410-03A_1x03_P2.54mm_Vertical, F.Cu at (317.4, 179.0)
- added ConnLIDAR1: ConnLIDAR, Connector_JST:JST_EH_B5B-EH-A_1x05_P2.50mm_Vertical, F.Cu at (188.8, 103.0)
- added ConnMotor1: ConnMotor1, Connector_JST:JST_EH_B6B-EH-A_1x06_P2.50mm_Vertical, F.Cu at (330.0, 91.8)
- added ConnMotor2: ConnMotor2, Connector_JST:JST_EH_B6B-EH-A_1x06_P2.50mm_Vertical, F.Cu at (330.0, 106.8)
- added ConnMotor3: ConnMotor3, Connector_JST:JST_EH_B6B-EH-A_1x06_P2.50mm_Vertical, F.Cu at (330.0, 121.8)
- added ConnNeoPixel1: ConnNeoPixel, Connector_Molex:Molex_KK-254_AE-6410-03A_1x03_P2.54mm_Vertical, F.Cu at (292.8, 151.8)
- added ConnPCA9685: ConnPCA9685, Connector_JST:JST_EH_B6B-EH-A_1x06_P2.50mm_Vertical, F.Cu at (141.4, 102.2)
- added ConnSerie1: ConnSerie, Connector_JST:JST_EH_B4B-EH-A_1x04_P2.50mm_Vertical, F.Cu at (165.1, 120.2)
- added ConnTirette1: ConnTirette, Connector_Molex:Molex_KK-254_AE-6410-02A_1x02_P2.54mm_Vertical, F.Cu at (166.2, 81.2)
- added G***: LOGO, LOGO, B.Cu at (295.0, 192.0)
- added G***: LOGO, LOGO, B.Cu at (295.0, 175.2)
- added R6: 110, Resistor_SMD:R_1206_3216Metric_Pad1.30x1.75mm_HandSolder, F.Cu at (310.0, 171.1)
- added R7: 470, Resistor_SMD:R_1206_3216Metric_Pad1.30x1.75mm_HandSolder, F.Cu at (313.2, 179.0)
- added R8: 110, Resistor_SMD:R_1206_3216Metric_Pad1.30x1.75mm_HandSolder, F.Cu at (310.0, 179.0)
- added connButton1: connButton1, Connector_Molex:Molex_KK-254_AE-6410-02A_1x02_P2.54mm_Vertical, F.Cu at (166.2, 72.3)
- C1, C2: footprint Capacitor_THT:CP_Radial_D5.0mm_P2.50mm -> Capacitor_THT:CP_Radial_D8.0mm_P3.50mm
- C3: footprint Capacitor_THT:CP_Radial_D8.0mm_P3.80mm -> Capacitor_THT:CP_Radial_D8.0mm_P3.50mm
- J1: value Conn_01x02 -> Conn_01x05; footprint Connector_JST:JST_XH_B2B-XH-A_1x02_P2.50mm_Vertical -> Connector_JST:JST_XH_B5B-XH-A_1x05_P2.50mm_Vertical
- R1, R2: value R -> 4,7k
- R3, R5: value R_Small -> 470
- R4: value R_Small -> 110
- U1: value TSR_2-2450 -> ESP32-S3-DevKitC; footprint Traco:Traco 2- 24xx -> PCM_Espressif:ESP32-S3-DevKitC
- moved H4 450.0 mm to (330.0, 200.0)
- moved R5 370.6 mm to (313.2, 171.1)
- moved C3 360.4 mm to (330.0, 98.8), turned to 180 degrees
- moved C1 332.2 mm to (330.0, 128.8), turned to 180 degrees
- moved H3 326.1 mm to (260.0, 200.0)
- moved R3 326.0 mm to (313.2, 163.3), turned to 90 degrees
- moved R4 322.0 mm to (310.0, 163.3), turned to -90 degrees
- moved C2 315.2 mm to (330.0, 113.8)
- moved H1 308.3 mm to (260.0, 80.0)
- moved U1 297.0 mm to (306.4, 137.3), turned to 180 degrees
- moved H2 285.5 mm to (330.0, 80.0)
- moved R1 200.2 mm to (158.6, 107.1), turned to 0 degrees
- moved R2 199.3 mm to (158.6, 110.4), turned to 0 degrees
- moved J1 177.8 mm to (160.9, 89.8)
Connections:
- C1 pad 1: +12V -> +BATT
- C2 pad 1: +5V -> +BATT
- C3 pad 1: +12V -> +BATT
- J1 pad 1: /GP2 -> GND
- J1 pad 2: GND -> Net-(J1-Pin_2)
- R3 pad 1: +3.3VP -> Net-(ConnIFM_1-Pin_1)
- R3 pad 2: Net-(D1-A) -> IFM1
- R4 pad 1: +5V -> IFM1
- R4 pad 2: Net-(D3-A) -> GND
- R5 pad 1: +12V -> Net-(ConnIFM_2-Pin_1)
- R5 pad 2: Net-(D4-A) -> IFM2
- U1 pad 1: +12V -> +3.3V
- U1 pad 2: GND -> +3.3V
- U1 pad 3: +5V -> unconnected-(U1-CHIP_PU-Pad3)
Routing:
- net +5V: track 284.4 -> 0.00 mm
- net +12V: track 214.2 -> 25.5 mm
- net +3.3VP: track 116.5 -> 0.00 mm, vias 1 -> 0
- net EN: track 135.2 -> 47.3 mm
- net SDA: track 87.0 -> 0.00 mm
- net SCL: track 86.9 -> 0.00 mm
- net +5VP: track 70.2 -> 0.00 mm
- net DIR3: track 58.2 -> 26.4 mm
- net STEP3: track 58.3 -> 30.5 mm
- net DIR1: track 36.2 -> 11.1 mm
- net +3.3V: track 24.5 -> 0.00 mm
- net STEP1: track 36.9 -> 14.7 mm
- net DIR2: track 39.7 -> 17.7 mm
- net GND: track 18.6 -> 0.00 mm, vias 3 -> 0
- net STEP2: track 39.7 -> 22.0 mm
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- added copper zone on F.Cu, net +BATT
- removed copper zone on B.Cu, net GND
- removed copper zone on F.Cu, net GND
Other:
- board outline removed
- board text added: "locked"
- board text removed: "Unimakers CDR 2024 Looij Dylan V0.3"

Commit message: Modified board
Parts:
- removed J1: Conn_01x05, Connector_JST:JST_XH_B5B-XH-A_1x05_P2.50mm_Vertical
- ConnBATT1: moved to B.Cu
- moved ConnI2C1 215.4 mm to (330.5, 160.2), turned to 180 degrees
- moved Conn5VL1 201.8 mm to (319.2, 160.2), turned to 180 degrees
- moved ConnAfficheur1 194.6 mm to (316.9, 169.0)
- moved ConnPCA9685 190.8 mm to (316.9, 177.2)
- moved Conn5V1 184.5 mm to (316.9, 86.5), turned to 90 degrees
- moved Conn5VP1 178.0 mm to (326.8, 184.8), turned to -90 degrees
- moved R2 158.0 mm to (315.0, 133.2), turned to 90 degrees
- moved R1 153.5 mm to (309.9, 133.2), turned to 90 degrees
- moved ConnButton3 114.1 mm to (269.2, 101.6), turned to 180 degrees
- moved ConnButton2 107.8 mm to (269.2, 94.0), turned to 180 degrees
- moved ConnTirette1 106.8 mm to (269.2, 109.2), turned to 180 degrees
- moved ConnSerie1 105.2 mm to (269.2, 134.8), turned to 90 degrees
- moved connButton1 104.0 mm to (269.2, 86.4), turned to 180 degrees
- moved ConnLIDAR1 94.0 mm to (269.2, 151.5), turned to 90 degrees
- moved ConnIFM_1 52.5 mm to (270.6, 187.0), turned to 90 degrees
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Connections:
- U1 pad 28: unconnected-(U1-GPIO47-Pad28) -> logique2
- U1 pad 29: SERVO_ENABLE -> logique3
- U1 pad 30: IFM2 -> Tirette
- U1 pad 32: logique2 -> unconnected-(U1-GPIO35-Pad32)
- U1 pad 33: logique3 -> SERVO_ENABLE
- U1 pad 34: Tirette -> IFM2
- U1 pad 36: Net-(J1-Pin_5) -> unconnected-(U1-GPIO39/MTCK-Pad36)
- U1 pad 37: Net-(J1-Pin_4) -> unconnected-(U1-GPIO40/MTDO-Pad37)
- U1 pad 38: Net-(J1-Pin_3) -> unconnected-(U1-GPIO41/MTDI-Pad38)
- U1 pad 39: Net-(J1-Pin_2) -> unconnected-(U1-GPIO42/MTMS-Pad39)
- U1 pad 41: unconnected-(U1-GPIO1/ADC1_CH0-Pad41) -> Neopixel
Routing:
- net SDA: track 0.00 -> 29.9 mm
- net SCL: track 0.00 -> 23.8 mm
- net logique1: track 0.00 -> 17.6 mm
- net Tirette: track 0.00 -> 17.4 mm
- net logique2: track 0.00 -> 15.5 mm
- net logique3: track 0.00 -> 15.3 mm
- net SERIAL_TX: track 0.00 -> 14.3 mm
- net SERIAL_RX: track 0.00 -> 14.3 mm
- net +5V: track 0.00 -> 10.5 mm
- net +5VL: track 0.00 -> 8.79 mm
- net +3.3V: track 0.00 -> 5.99 mm
- net STEP2: track 22.0 -> 19.1 mm
- net STEP3: track 30.5 -> 27.7 mm
- net DIR2: track 17.7 -> 15.5 mm
- net DIR3: track 26.4 -> 24.2 mm
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- added copper zone on F.Cu, net +5VP
- added copper zone on B.Cu, net +BATT
- added copper zone on B.Cu, net GND
- added copper zone on F.Cu, net GND
Other:
- board outline added: 82 x 132 mm
