File: MainBoardV3/MainboardV3.kicad_sch (KiCad schematic)
At the start: 38 parts, among them U1 ESP32-S3-DevKitC, U2 ESP32-S3

Commit message: Modified board
Parts:
- removed U2: ESP32-S3, Package_DFN_QFN:QFN-56-1EP_7x7mm_P0.4mm_EP5.6x5.6mm, symbol PCM_Espressif:ESP32-S3
- renumbered ConnAfficheur to ConnAfficheur1, ConnSerie to ConnSerie1
Connections:
- net IFM2: now also U1.34 (GPIO37); no longer U1.30 (GPIO45)
- net Neopixel: now also U1.41 (GPIO1/ADC1_CH0)
- net SERVO_ENABLE: now also U1.33 (GPIO36); no longer U1.29 (GPIO48)
- net Tirette: now also U1.30 (GPIO45); no longer U1.34 (GPIO37)
- net logique2: now also U1.28 (GPIO47); no longer U1.32 (GPIO35)
- net logique3: now also U1.29 (GPIO48); no longer U1.33 (GPIO36)
Changed lines of the file:
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@@
   (junction (at 260.35 129.54) (diameter 0) (color 0 0 0 0)
   )
-  (junction (at 209.55 151.13) (diameter 0) (color 0 0 0 0)
-  )
   (junction (at 125.73 149.86) (diameter 0) (color 0 0 0 0)
   )
@@
     (stroke (width 0) (type default))
   )
-  (wire (pts (xy 209.55 149.86) (xy 209.55 151.13))
-    (stroke (width 0) (type default))
-  )
   (wire (pts (xy 156.21 132.08) (xy 167.64 132.08))
     (stroke (width 0) (type default))
@@
     (stroke (width 0) (type default))
   )
+  (wire (pts (xy 209.55 149.86) (xy 209.55 152.4))
+    (stroke (width 0) (type default))
+  )
   (wire (pts (xy 165.1 149.86) (xy 165.1 152.4))
     (stroke (width 0) (type default))
@@
   )
   (wire (pts (xy 34.29 81.28) (xy 33.02 81.28))
-    (stroke (width 0) (type default))
-  )
-  (wire (pts (xy 209.55 152.4) (xy 209.55 151.13))
     (stroke (width 0) (type default))
   )
@@
     (effects (font (size 1.27 1.27)) (justify right bottom))
   )
-  (label "GP1" (at 131.445 49.53 0) (fields_autoplaced)
+  (label "GP1" (at 144.78 48.26 0) (fields_autoplaced)
     (effects (font (size 1.27 1.27)) (justify left bottom))
   )
-  (label "GP2" (at 131.445 52.07 0) (fields_autoplaced)
+  (label "GP2" (at 144.78 52.07 0) (fields_autoplaced)
     (effects (font (size 1.27 1.27)) (justify left bottom))
   )
@@
     )
   )
+  (global_label "Neopixel" (shape output) (at 130.81 49.53 0) (fields_autoplaced)
+    (effects (font (size 1.27 1.27)) (justify left))
+    (property "Intersheetrefs" "${INTERSHEET_REFS}" (at 141.899 49.53 0)
+      (effects (font (size 1.27 1.27)) (justify left) hide)
+    )
+  )
   (global_label "SCL" (shape input) (at 251.46 113.03 180) (fields_autoplaced)
     (effects (font (size 1.27 1.27)) (justify right))
@@
     )
   )
+  (global_label "logique2" (shape input) (at 130.81 107.95 0) (fields_autoplaced)
+    (effects (font (size 1.27 1.27)) (justify left))
+    (property "Intersheetrefs" "${INTERSHEET_REFS}" (at 140.2765 107.95 0)
+      (effects (font (size 1.27 1.27)) (justify left) hide)
+    )
+  )
   (global_label "SDA" (shape input) (at 251.46 110.49 180) (fields_autoplaced)
     (effects (font (size 1.27 1.27)) (justify right))
@@
     )
   )
-  (global_label "logique2" (shape input) (at 130.81 92.71 0) (fields_autoplaced)
-    (effects (font (size 1.27 1.27)) (justify left))
-    (property "Intersheetrefs" "${INTERSHEET_REFS}" (at 140.2765 92.71 0)
-      (effects (font (size 1.27 1.27)) (justify left) hide)
-    )
-  )
-  (global_label "IFM2" (shape input) (at 130.81 102.87 0) (fields_autoplaced)
-    (effects (font (size 1.27 1.27)) (justify left))
-    (property "Intersheetrefs" "${INTERSHEET_REFS}" (at 137.3757 102.87 0)
+  (global_label "IFM2" (shape input) (at 130.81 97.79 0) (fields_autoplaced)
+    (effects (font (size 1.27 1.27)) (justify left))
+    (property "Intersheetrefs" "${INTERSHEET_REFS}" (at 137.3757 97.79 0)
       (effects (font (size 1.27 1.27)) (justify left) hide)
     )
@@
     )
   )
-  (global_label "SERVO_ENABLE" (shape input) (at 130.81 110.49 0) (fields_autoplaced)
-    (effects (font (size 1.27 1.27)) (justify left))
-    (property "Intersheetrefs" "${INTERSHEET_REFS}" (at 146.4778 110.49 0)
+  (global_label "SERVO_ENABLE" (shape input) (at 130.81 95.25 0) (fields_autoplaced)
+    (effects (font (size 1.27 1.27)) (justify left))
+    (property "Intersheetrefs" "${INTERSHEET_REFS}" (at 146.4778 95.25 0)
       (effects (font (size 1.27 1.27)) (justify left) hide)
     )
@@
     )
   )
-  (global_label "Tirette" (shape input) (at 130.81 97.79 0) (fields_autoplaced)
-    (effects (font (size 1.27 1.27)) (justify left))
-    (property "Intersheetrefs" "${INTERSHEET_REFS}" (at 138.6797 97.79 0)
+  (global_label "Tirette" (shape input) (at 130.81 102.87 0) (fields_autoplaced)
+    (effects (font (size 1.27 1.27)) (justify left))
+    (property "Intersheetrefs" "${INTERSHEET_REFS}" (at 138.6797 102.87 0)
       (effects (font (size 1.27 1.27)) (justify left) hide)
     )
@@
     )
   )
-  (global_label "logique3" (shape input) (at 130.81 95.25 0) (fields_autoplaced)
-    (effects (font (size 1.27 1.27)) (justify left))
-    (property "Intersheetrefs" "${INTERSHEET_REFS}" (at 140.2976 95.25 0)
+  (global_label "logique3" (shape input) (at 130.81 110.49 0) (fields_autoplaced)
+    (effects (font (size 1.27 1.27)) (justify left))
+    (property "Intersheetrefs" "${INTERSHEET_REFS}" (at 140.2976 110.49 0)
       (effects (font (size 1.27 1.27)) (justify left) hide)
     )
@@
   (symbol (lib_id "Connector_Generic:Conn_01x04") (at 256.54 148.59 0) (unit 1)
     (in_bom yes) (on_board yes) (dnp no) (fields_autoplaced)
-    (property "Reference" "ConnSerie" (at 259.08 148.5899 0)
+    (property "Reference" "ConnSerie1" (at 259.08 148.5899 0)
       (effects (font (size 1.27 1.27)) (justify left))
     )
@@
       (project "MainboardV3"
         (path "/ccdda621-e361-4147-9a57-71374655ba08"
-          (reference "ConnSerie") (unit 1)
+          (reference "ConnSerie1") (unit 1)
         )
       )
@@
     )
   )
-  (symbol (lib_id "power:GND") (at 209.55 151.13 0) (unit 1)
+  (symbol (lib_id "power:GND") (at 209.55 152.4 0) (unit 1)
     (in_bom yes) (on_board yes) (dnp no)
-    (property "Reference" "#PWR078" (at 209.55 157.48 0)
-      (effects (font (size 1.27 1.27)) hide)
-    )
-    (property "Value" "GND" (at 212.09 153.6699 0)
-      (effects (font (size 1.27 1.27)) (justify left))
-    )
-    (property "Footprint" "" (at 209.55 151.13 0)
-      (effects (font (size 1.27 1.27)) hide)
-    )
-    (property "Datasheet" "" (at 209.55 151.13 0)
+    (property "Reference" "#PWR078" (at 209.55 158.75 0)
+      (effects (font (size 1.27 1.27)) hide)
+    )
+    (property "Value" "GND" (at 212.09 154.9399 0)
+      (effects (font (size 1.27 1.27)) (justify left))
+    )
+    (property "Footprint" "" (at 209.55 152.4 0)
+      (effects (font (size 1.27 1.27)) hide)
+    )
+    (property "Datasheet" "" (at 209.55 152.4 0)
       (effects (font (size 1.27 1.27)) hide)
     )
@@
     )
   )
-  (symbol (lib_id "PCM_Espressif:ESP32-S3") (at -39.37 58.42 0) (unit 1)
-    (in_bom yes) (on_board yes) (dnp no) (fields_autoplaced)
-    (property "Reference" "U2" (at -37.1459 99.06 0)
-      (effects (font (size 1.27 1.27)) (justify left))
-    )
-    (property "Value" "ESP32-S3" (at -37.1459 101.6 0)
-      (effects (font (size 1.27 1.27)) (justify left))
-    )
-    (property "Footprint" "Package_DFN_QFN:QFN-56-1EP_7x7mm_P0.4mm_EP5.6x5.6mm" (at -39.37 106.68 0)
-      (effects (font (size 1.27 1.27)) hide)
-    )
-    (property "Datasheet" "https://www.espressif.com/sites/default/files/documentation/esp32-s3_datasheet_en.pdf" (at -39.37 109.22 0)
-      (effects (font (size 1.27 1.27)) hide)
-    )
-    (pin "36")
-    (pin "37")
-    (pin "1")
-    (pin "10")
-    (pin "11")
-    (pin "12")
-    (pin "13")
-    (pin "14")
-    (pin "15")
-    (pin "16")
-    (pin "17")
-    (pin "18")
-    (pin "19")
-    (pin "2")
-    (pin "20")
-    (pin "21")
-    (pin "22")
-    (pin "23")
-    (pin "24")
-    (pin "25")
-    (pin "26")
-    (pin "27")
-    (pin "28")
-    (pin "29")
-    (pin "3")
-    (pin "30")
-    (pin "31")
-    (pin "32")
-    (pin "33")
-    (pin "34")
-    (pin "35")
-    (pin "38")
-    (pin "39")
-    (pin "4")
-    (pin "40")
-    (pin "41")
-    (pin "42")
-    (pin "43")
-    (pin "44")
-    (pin "45")
-    (pin "46")
-    (pin "47")
-    (pin "48")
-    (pin "49")
-    (pin "5")
-    (pin "50")
-    (pin "51")
-    (pin "52")
-    (pin "53")
-    (pin "54")
-    (pin "55")
-    (pin "56")
-    (pin "57")
-    (pin "6")
-    (pin "7")
-    (pin "8")
-    (pin "9")
-    (instances
-      (project "MainboardV3"
-        (path "/ccdda621-e361-4147-9a57-71374655ba08"
-          (reference "U2") (unit 1)
-        )
-      )
-    )
-  )
   (symbol (lib_id "Device:R") (at 256.54 127 270) (unit 1)
     (in_bom yes) (on_board yes) (dnp no) (fields_autoplaced)
@@
   (symbol (lib_id "Connector_Generic:Conn_01x06") (at 209.55 118.11 180) (unit 1)
     (in_bom yes) (on_board yes) (dnp no) (fields_autoplaced)
-    (property "Reference" "ConnAfficheur" (at 209.55 104.14 0)
+    (property "Reference" "ConnAfficheur1" (at 209.55 104.14 0)
       (effects (font (size 1.27 1.27)))
     )
@@
       (project "MainboardV3"
         (path "/ccdda621-e361-4147-9a57-71374655ba08"
-          (reference "ConnAfficheur") (unit 1)
-        )
-      )
+          (reference "ConnAfficheur1") (unit 1)
+        )
+      )
